Commit message: using base_link instead, got somewhere with planner but keeps cutting between cones. might have to use boundary interp

File: sam_bot_description/src/description/sam_bot_description.urdf (robot description, URDF)
Before this commit: robot sam_bot, 7 links, 6 joints
Links:
- removed link base_footprint
- added link base_link
Joints:
- joint base_joint: child base_footprint -> base_link
